File: KiCAD Files/Rev01/VideoULA.kicad_pcb (KiCad board)
At the start: 2 copper layers, 17.8 x 35.6 mm, 19 parts, among them IC6 VC2069 Socket, J1 JTAG-IDC, J2 Conn_01x01, U1 XC9572XL-10VQG44C, U2 XC6206P332MR, U3 IS62C256AL, X1 48MHz

Commit message: Updated value of C7 & C8
Parts:
- C7, C8: value 10n -> 10u
