File: KiCAD Files/Rev01/VideoULA.kicad_sch (KiCad schematic)
At the start: 19 parts, among them IC6 VC2069 Socket, J1 JTAG-IDC, J2 Conn_01x01, U1 XC9572XL-10VQG44C, U2 XC6206P332MR, U3 IS62C256AL, X1 48MHz

Commit message: Updated value of C7 & C8
Parts:
- C7, C8: value 10n -> 10u; JLC Part Number C57112 -> C19702
Changed lines of the file:
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@@
 	(title_block
 		(title "Model B - Video ULA Replacement")
-		(date "2026-07-13")
-		(rev "01")
+		(date "2026-08-07")
+		(rev "01a")
 		(company "Ken Lowe")
-		(comment 1 "Rev 01: Initial Release. Final issue swaps / fixes ULA R/R_in & B/B_in pin assignment")
+		(comment 1 "Rev01a: Change C7 and C8 from 10nF to 10uF")
+		(comment 2 "Rev 01: Initial Release. Final issue swaps / fixes ULA R/R_in & B/B_in pin assignment")
 	)
 	(junction
@@
 			)
 		)
-		(property "Datasheet" "https://jlc-prod-smt.oss-eu-central-1.aliyuncs.com/smtDataManualFile/8667086713656442880-C14663.pdf"
+		(property "Datasheet" ""
 			(at 25.4 115.57 0)
 			(hide yes)
@@
 			)
 		)
-		(property "Datasheet" "https://jlc-prod-smt.oss-eu-central-1.aliyuncs.com/smtDataManualFile/8579707861616033792-C5446.pdf"
+		(property "Datasheet" ""
 			(at 39.37 67.31 0)
 			(hide yes)
@@
 			)
 		)
-		(property "Datasheet" "https://jlc-prod-smt.oss-eu-central-1.aliyuncs.com/smtDataManualFile/8667086713656442880-C14663.pdf"
+		(property "Datasheet" ""
 			(at 57.15 115.57 0)
 			(hide yes)
@@
 			)
 		)
-		(property "Datasheet" "https://jlc-prod-smt.oss-eu-central-1.aliyuncs.com/smtDataManualFile/8556213788455567360-C15849.pdf"
+		(property "Datasheet" ""
 			(at 25.4 71.12 0)
 			(hide yes)
@@
 			)
 		)
-		(property "Value" "10n"
+		(property "Value" "10u"
 			(at 37.8968 116.713 0)
 			(show_name no)
@@
 			)
 		)
-		(property "Datasheet" "https://jlc-prod-smt.oss-eu-central-1.aliyuncs.com/smtDataManualFile/8757265887555018752-C57112.pdf"
+		(property "Datasheet" ""
 			(at 35.56 115.57 0)
 			(hide yes)
@@
 			)
 		)
-		(property "JLC Part Number" "C57112"
+		(property "JLC Part Number" "C19702"
 			(at 35.56 115.57 0)
 			(hide yes)
@@
 			)
 		)
-		(property "Datasheet" "https://jlc-prod-smt.oss-eu-central-1.aliyuncs.com/smtDataManualFile/8579706381316128768-C25804.pdf"
+		(property "Datasheet" ""
 			(at 107.95 119.38 0)
 			(hide yes)
@@
 			)
 		)
-		(property "Datasheet" "https://jlc-prod-smt.oss-eu-central-1.aliyuncs.com/smtDataManualFile/8590164980525142016-C454614.pdf"
+		(property "Datasheet" ""
 			(at 36.83 36.83 0)
 			(hide yes)
@@
 			)
 		)
-		(property "Datasheet" "https://jlc-prod-smt.oss-eu-central-1.aliyuncs.com/smtDataManualFile/8588914457561485312-C569042.pdf"
+		(property "Datasheet" ""
 			(at 127 67.31 0)
 			(hide yes)
@@
 			)
 		)
-		(property "Datasheet" "https://jlc-prod-smt.oss-eu-central-1.aliyuncs.com/smtDataManualFile/8579705779290898432-C29718.pdf"
+		(property "Datasheet" ""
 			(at 251.46 53.34 0)
 			(hide yes)
@@
 			)
 		)
-		(property "Datasheet" "https://jlc-prod-smt.oss-eu-central-1.aliyuncs.com/smtDataManualFile/8667086713656442880-C14663.pdf"
+		(property "Datasheet" ""
 			(at 25.4 93.98 0)
 			(hide yes)
@@
 			)
 		)
-		(property "Datasheet" "https://jlc-prod-smt.oss-eu-central-1.aliyuncs.com/smtDataManualFile/8667086713656442880-C14663.pdf"
+		(property "Datasheet" ""
 			(at 45.72 93.98 0)
 			(hide yes)
@@
 			)
 		)
-		(property "Datasheet" "https://jlc-prod-smt.oss-eu-central-1.aliyuncs.com/smtDataManualFile/8556213788455567360-C15849.pdf"
+		(property "Datasheet" ""
 			(at 52.07 71.12 0)
 			(hide yes)
@@
 			)
 		)
-		(property "Datasheet" "https://jlc-prod-smt.oss-eu-central-1.aliyuncs.com/smtDataManualFile/8588881829030346752-C47143.pdf"
+		(property "Datasheet" ""
 			(at 214.63 49.53 0)
 			(hide yes)
@@
 			)
 		)
-		(property "Value" "10n"
+		(property "Value" "10u"
 			(at 49.3268 116.713 0)
 			(show_name no)
@@
 			)
 		)
-		(property "Datasheet" "https://jlc-prod-smt.oss-eu-central-1.aliyuncs.com/smtDataManualFile/8757265887555018752-C57112.pdf"
+		(property "Datasheet" ""
 			(at 46.99 115.57 0)
 			(hide yes)
@@
 			)
 		)
-		(property "JLC Part Number" "C57112"
+		(property "JLC Part Number" "C19702"
 			(at 46.99 115.57 0)
 			(hide yes)
@@
 			)
 		)
-		(property "Datasheet" "https://jlc-prod-smt.oss-eu-central-1.aliyuncs.com/smtDataManualFile/8667086713656442880-C14663.pdf"
+		(property "Datasheet" ""
 			(at 35.56 93.98 0)
 			(hide yes)
